Commit message: feat: robot physically drives to stations in Gazebo (V4 navigation)

File: ros2_ws/src/ai_robot/models/ai_robot.urdf (robot description, URDF)
Before this commit: robot ai_robot, 4 links, 3 joints
Links:
- added link caster_back_link, mass 0.1; collision sphere radius=0.05; visual sphere radius=0.05
- added link caster_link, mass 0.1; collision sphere radius=0.05; visual sphere radius=0.05
Joints:
- added joint caster_back_joint: type fixed, parent base_link, child caster_back_link
- added joint caster_joint: type fixed, parent base_link, child caster_link
